Commit message: Actualización nombre paquete

File: urdf/px.urdf (robot description, URDF)
Before this commit: robot px_robot, 7 links, 6 joints
Links:
- link base_link: geometry visual mesh filename=package://px_robot_CV/meshes/Base.STL scale=1 1 1
- link link1: geometry visual mesh filename=package://px_robot_CV/meshes/Shoulder.STL scale=1 1 1
- link link2: geometry visual mesh filename=package://px_robot_CV/meshes/Bicep.STL scale=1 1 1
- link link3: geometry visual mesh filename=package://px_robot_CV/meshes/Bicep.STL scale=1 1 1
- link link4: geometry visual mesh filename=package://px_robot_CV/meshes/Wrist.STL scale=1 1 1

Commit message: Ajuste name pkg y modelo URDF

File: urdf/px.urdf (robot description, URDF)
Before this commit: robot px_robot_CV, 7 links, 6 joints
Joints:
- joint joint_1: origin xyz=0.0 0.0 0.09 rpy=0.0 0.0 0.0 -> xyz=0.0 0.0 0.09 rpy=0.0 0.0 3.141592
- joint joint_2: origin xyz=0.0 0.0 0.042 rpy=1.5707 0.0 0.0 -> xyz=0.0 0.0 0.047 rpy=-1.5707 0.0 0.0
- joint joint_3: origin xyz=0.0 0.1065 0 rpy=0.0 0.0 0.0 -> xyz=0.032 -0.100 0 rpy=0.0 0.0 -1.2611
- joint joint_4: origin xyz=0.0 0.1065 0 rpy=0.0 0.0 0.0 -> xyz=0.095242 -0.030478 0 rpy=0.0 0.0 -0.3097
- joint tcp: origin xyz=0.0 0.092 0 rpy=-1.5707 0.0 0.0 -> xyz=0.100 0.0 0 rpy=1.5707 0.0 1.5707

File: urdf/px_collision.urdf (robot description, URDF)
Before this commit: robot px_robot, 7 links, 6 joints
Links:
- link base_link: geometry collision mesh filename=package://px_robot_CV/meshes/Base.STL scale=1 1 1; visual mesh filename=package://px_robot_CV/meshes/Base.STL scale=1 1 1
- link link1: geometry collision mesh filename=package://px_robot_CV/meshes/Shoulder.STL scale=1 1 1; visual mesh filename=package://px_robot_CV/meshes/Shoulder.STL scale=1 1 1
- link link2: geometry collision mesh filename=package://px_robot_CV/meshes/Bicep.STL scale=1 1 1; visual mesh filename=package://px_robot_CV/meshes/Bicep.STL scale=1 1 1
- link link3: geometry collision mesh filename=package://px_robot_CV/meshes/Bicep.STL scale=1 1 1; visual mesh filename=package://px_robot_CV/meshes/Bicep.STL scale=1 1 1
- link link4: geometry collision mesh filename=package://px_robot_CV/meshes/Wrist.STL scale=1 1 1; visual mesh filename=package://px_robot_CV/meshes/Wrist.STL scale=1 1 1

File: urdf/px_transmission.urdf (robot description, URDF)
Before this commit: robot px_robot, 7 links, 6 joints
Links:
- link base_link: geometry visual mesh filename=package://px_robot_CV/meshes/Base.STL scale=1 1 1
- link link1: geometry visual mesh filename=package://px_robot_CV/meshes/Shoulder.STL scale=1 1 1
- link link2: geometry visual mesh filename=package://px_robot_CV/meshes/Bicep.STL scale=1 1 1
- link link3: geometry visual mesh filename=package://px_robot_CV/meshes/Bicep.STL scale=1 1 1
- link link4: geometry visual mesh filename=package://px_robot_CV/meshes/Wrist.STL scale=1 1 1

Commit message: Cambio final URDF modelo nuevo

File: urdf/px.urdf (robot description, URDF)
Before this commit: robot px_robot_CV, 7 links, 6 joints
Links:
- link base_link: geometry visual mesh filename=package://px_robot_CV/meshes/PX100_Base.stl scale=0.001 0.001 0.001
- link link1: geometry visual mesh filename=package://px_robot_CV/meshes/PX100_Shoulder.stl scale=0.001 0.001 0.001
- link link2: geometry visual mesh filename=package://px_robot_CV/meshes/PX100_Bicep.stl scale=0.001 0.001 0.001
- link link3: geometry visual mesh filename=package://px_robot_CV/meshes/PX100_Forearm.stl scale=0.001 0.001 0.001
- link link4: geometry visual mesh filename=package://px_robot_CV/meshes/PX100_Wrist.stl scale=0.001 0.001 0.001
Joints:
- joint joint_1: origin xyz=0.0 0.0 0.09 rpy=0.0 0.0 3.141592 -> xyz=0.0 0.0 0.049 rpy=0.0 0.0 3.141592

Commit message: Cambios URDF orientacón Z

File: urdf/px.urdf (robot description, URDF)
Before this commit: robot px_robot_CV, 7 links, 6 joints
Joints:
- joint joint_3: origin xyz=0.032 -0.100 0 rpy=0.0 0.0 -1.2611 -> xyz=0.032 -0.100 0 rpy=3.141592 0.0 -1.2611
- joint joint_4: origin xyz=0.095242 -0.030478 0 rpy=0.0 0.0 -0.3097 -> xyz=0.095242 -0.030478 0 rpy=3.141592 0.0 -0.3097

Commit message: Mas cambios URDF

File: urdf/px.urdf (robot description, URDF)
Before this commit: robot px_robot_CV, 7 links, 6 joints
Joints:
- joint joint_1: origin xyz=0.0 0.0 0.049 rpy=0.0 0.0 3.141592 -> xyz=0.0 0.0 0.049 rpy=3.141592 0.0 3.141592
- joint joint_4: origin xyz=0.095242 -0.030478 0 rpy=3.141592 0.0 -0.3097 -> xyz=0.095242 -0.030478 0 rpy=-3.141592 0.0 -0.3097

Commit message: urdf

File: urdf/px.urdf (robot description, URDF)
Before this commit: robot px_robot_CV, 7 links, 6 joints
Joints:
- joint joint_1: origin xyz=0.0 0.0 0.049 rpy=3.141592 0.0 3.141592 -> xyz=0.0 0.0 0.049 rpy=0.0 0.0 3.141592

Commit message: URDF

File: urdf/px.urdf (robot description, URDF)
Before this commit: robot px_robot_CV, 7 links, 6 joints
Joints:
- joint joint_1: origin xyz=0.0 0.0 0.049 rpy=0.0 0.0 3.141592 -> xyz=0.0 0.0 0.049 rpy=3.141592 0.0 3.141592

Commit message: URDF

File: urdf/px.urdf (robot description, URDF)
Before this commit: robot px_robot_CV, 7 links, 6 joints
Joints:
- joint joint_1: origin xyz=0.0 0.0 0.049 rpy=3.141592 0.0 3.141592 -> xyz=0.0 0.0 0.049 rpy=1.5707 0.0 3.141592

Commit message: URDF

File: urdf/px.urdf (robot description, URDF)
Before this commit: robot px_robot_CV, 7 links, 6 joints
Joints:
- joint joint_1: origin xyz=0.0 0.0 0.049 rpy=1.5707 0.0 3.141592 -> xyz=0.0 0.0 0.049 rpy=0.0 0.0 3.141592
- joint joint_2: origin xyz=0.0 0.0 0.047 rpy=-1.5707 0.0 0.0 -> xyz=0.0 0.0 0.047 rpy=1.5707 0.0 0.0

Commit message: urdf

File: urdf/px.urdf (robot description, URDF)
Before this commit: robot px_robot_CV, 7 links, 6 joints
Joints:
- joint joint_3: origin xyz=0.032 -0.100 0 rpy=3.141592 0.0 -1.2611 -> xyz=0.032 0.100 0 rpy=3.141592 0.0 -1.2611

Commit message: URDF

File: urdf/px.urdf (robot description, URDF)
Before this commit: robot px_robot_CV, 7 links, 6 joints
Joints:
- joint joint_3: origin xyz=0.032 0.100 0 rpy=3.141592 0.0 -1.2611 -> xyz=0.032 0.100 0 rpy=0.0 0.0 -1.2611

Commit message: urdf

File: urdf/px.urdf (robot description, URDF)
Before this commit: robot px_robot_CV, 7 links, 6 joints
Joints:
- joint joint_3: origin xyz=0.032 0.100 0 rpy=0.0 0.0 -1.2611 -> xyz=0.032 0.100 0 rpy=0.0 0.0 0.3097

Commit message: URDF Ojala final

File: urdf/px.urdf (robot description, URDF)
Before this commit: robot px_robot_CV, 7 links, 6 joints
Joints:
- joint joint_4: origin xyz=0.095242 -0.030478 0 rpy=-3.141592 0.0 -0.3097 -> xyz=0.095242 -0.030478 0 rpy=0.0 0.0 -0.3097

Commit message: URDF final prometido

File: urdf/px.urdf (robot description, URDF)
Before this commit: robot px_robot_CV, 7 links, 6 joints
Joints:
- joint tcp: origin xyz=0.100 0.0 0 rpy=1.5707 0.0 1.5707 -> xyz=0.100 0.0 0 rpy=1.5707 0.0 -1.5707

Commit message: URDF

File: urdf/px.urdf (robot description, URDF)
Before this commit: robot px_robot_CV, 7 links, 6 joints
Joints:
- joint tcp: origin xyz=0.100 0.0 0 rpy=1.5707 0.0 -1.5707 -> xyz=0.100 0.0 0 rpy=-1.5707 0.0 -1.5707

Commit message: Sección 4

File: urdf/px.urdf (robot description, URDF)
Before this commit: robot px_robot_CV, 7 links, 6 joints
Joints:
- joint joint_3: origin xyz=0.032 0.100 0 rpy=0.0 0.0 0.3097 -> xyz=0.032 0.100 0 rpy=0.0 0.0 1.261094
- joint joint_4: origin xyz=0.095242 -0.030478 0 rpy=0.0 0.0 -0.3097 -> xyz=0.095242 0.030478 0 rpy=0.0 0.0 0.3097
